File: beaglebone_can_cape.kicad_pcb (KiCad board)
At the start: 2 copper layers, 86.4 x 54.6 mm, 6 parts, among them P8 BeagleBone_Black_Header, P9 BeagleBone_Black_Header

Commit message: finished sch, adding footprints now
Parts:
- added J1: DCAN0, TerminalBlock_RND:TerminalBlock_RND_205-00232_1x02_P5.08mm_Horizontal, F.Cu at (127.5, 63.6)
- added J2: DCAN1, TerminalBlock_RND:TerminalBlock_RND_205-00232_1x02_P5.08mm_Horizontal, F.Cu at (127.5, 74.4)
- added JP1: Jumper_2_Open, Connector_PinHeader_2.54mm:PinHeader_1x02_P2.54mm_Vertical, F.Cu at (148.5, 59.5)
- added JP2: Jumper_2_Open, Connector_PinHeader_2.54mm:PinHeader_1x02_P2.54mm_Vertical, F.Cu at (157.2, 62.8)
